File: hardware/stm32-tutorial-project/stm32-tutorial-project.kicad_pcb (KiCad board)
At the start: 2 copper layers, 7 parts, among them J2 10pin IDC SWD, U1 STM32G431CBTx

Commit message: removed anything in it to start anew
Parts:
- removed D11: SP0504BAHT, Package_TO_SOT_SMD:SOT-23-5
- removed D12: PTVS7V5Z1USK, Diode_SMD:Nexperia_DSN1608-2_1.6x0.8mm
- removed F1: Fuse, Fuse:Fuse_0805_2012Metric
- removed FB1, FB2: 220 OHM, Inductor_SMD:L_0603_1608Metric_Pad1.05x0.95mm_HandSolder
- removed J2: 10pin IDC SWD, Connector_IDC:IDC-Header_2x05_P2.54mm_Vertical
- removed U1: STM32G431CBTx, Package_QFP:LQFP-48_7x7mm_P0.5mm
